File: kicad/offline_board/offline_board.kicad_sch (KiCad schematic)
At the start: 16 parts, among them J1 5.5x2.5 5V, J2 Display, Q1 PMOS, SW1 POWER, U1 Raspberry Pi Zero 2 W

Commit message: Major part of schematic is already done
Parts:
- added C10, C8: 22u, symbol Device:C
- added C5: 2u2, symbol Device:C
- added C6, C7: 100n, symbol Device:C
- added C9: 47p, symbol Device:C
- added J3: charger_1, symbol Connector_Generic:Conn_01x02
- added J4: charger_2, symbol Connector_Generic:Conn_01x02
- added L1: 2u2, symbol Device:L_Ferrite
- added Q2, Q5: DMP3007LSS-13, Package_SO:SOIC-8_3.9x4.9mm_P1.27mm, symbol Transistor_FET:FDS9435A
- added Q3, Q4: 2N7002, Package_TO_SOT_SMD:SOT-23, symbol Transistor_FET:2N7002
- added R10, R7: 100k, symbol Device:R
- added R11, R6: 10k, symbol Device:R
- added R4: 246k, symbol Device:R
- added R5: 47k, symbol Device:R
- added R8, R9: 100, symbol Device:R
- added SW2: 1, symbol Switch:SW_Push
- added SW3: 2, symbol Switch:SW_Push
- added SW4: 3, symbol Switch:SW_Push
- added SW5: 4, symbol Switch:SW_Push
- J1: value 5.5x2.5 5V -> 5.5x2.5 12V
Connections:
- net +5V: now also C10.1, C8.1, C9.1, L1.1, R4.2
- net 12V: now also U2.1 (EN), U2.3 (SUP), C5.1, C6.2, Q2.1 (S), Q2.2 (S), Q2.3 (S), Q5.1 (S), Q5.2 (S), Q5.3 (S), R11.2, R6.2
- net GND: now also C10.2, C5.2, C6.1, C8.2, J3.2 (Pin_2), J4.2 (Pin_2), Q3.2 (S), Q4.2 (S), R10.1, R5.1, R7.1, SW2.1, SW3.1, SW4.1, SW5.1
- net GPIO5: now reaches U1.29 (GPIO5)
- net GPIO5: now also SW5.2
- net GPIO6: now reaches U1.31 (GPIO6)
- net GPIO6: now also SW4.2
- net GPIO13: now reaches U1.33 (GPIO13)
- net GPIO13: now also SW3.2
- net GPIO19: now reaches U1.35 (GPIO19)
- net GPIO19: now also SW2.2
- net CH_2: now reaches U1.38 (GPIO20)
- net CH_2: now also R9.1
- net CH_1: now reaches U1.40 (GPIO21)
- net CH_1: now also R8.1
- net FB: now reaches U2.13 (FB)
- net FB: now also C9.2, R4.1, R5.2
- net at U2.5 (LX): now also C7.2, L1.2
- net at U2.9 (BST): now also C7.1
- new net: Q4.1 (G), R10.2, R9.2
- new net: Q3.1 (G), R7.2, R8.2
- new net: Q4.3 (D), Q5.4 (G), R11.1
- new net: J4.1 (Pin_1), Q5.5 (D), Q5.6 (D), Q5.7 (D), Q5.8 (D)
- new net: J3.1 (Pin_1), Q2.5 (D), Q2.6 (D), Q2.7 (D), Q2.8 (D)
- new net: Q2.4 (G), Q3.3 (D), R6.1
Other:
- note added: "TODO: perform logic conversion for led"
- moved on the sheet: C2, C3, C4, J2, R2, R3, U2
